File: pcb/pcb.kicad_pcb (KiCad board)
At the start: 2 copper layers, 228.6 x 86.5 mm, 121 parts, among them J1 USB_C_Receptacle_USB2.0, SW1 RST, SW2 RST, U1 USBLC6-2SC6, U2 STM32F072C8Tx, U3 XC6206PxxxMR-Regulator_Linear

Commit message: Add proper readme
Parts:
- added G***: LOGO, masonry.prety:logo_lg, F.Cu at (71.1, 64.4)
Other:
- board text added: "Masonry PCB"
- board text added: "Rev 1 designed by dcpedit github.com/dcpedit/masonry"
